File: circuit/adapter/adapter.sch (KiCad schematic (older format))
At the start: 15 parts, among them IC1 ATMEGA8-P, IC10 ATTINY84-P, IC2 ATTINY2313-P, IC3 ATMEGA16-P, IC4 ATTINY26-P, IC5 AT90S8515-P, IC7 ATTINY15-P-GOOD, IC8 ATTINY11-P, IC9 ATMEGA16M1-M, P1 CONN_10X2

Commit message: adapter PCB: open with Kicad 4.x and saving
Parts:
- C2, C3, C4, C5, C6: symbol CPSMALL -> CPsmall
- IC2: symbol ATTINY2313-P -> ATTINY2313-P-RESCUE-adapter
- IC4: symbol ATTINY26-P -> ATTINY26-P-RESCUE-adapter
- IC5: symbol AT90S8515-P -> AT90S8515-P-RESCUE-adapter
- IC7: symbol ATTINY15-P-GOOD -> ATTINY15-P-good
- IC8: symbol ATTINY11-P -> ATTINY11-P-RESCUE-adapter
Changed lines of the file:
@@
-EESchema Schematic File Version 2  date Čet 30 Kol 2012 17:04:33
+EESchema Schematic File Version 2
+LIBS:adapter-rescue
 LIBS:power
 LIBS:device
@@
 LIBS:memory
 LIBS:xilinx
-LIBS:special
 LIBS:microcontrollers
 LIBS:dsp
@@
 LIBS:attiny15-p-good
 LIBS:adapter-cache
-EELAYER 25  0
+EELAYER 25 0
 EELAYER END
-$Descr A3 16535 11700
+$Descr A3 16535 11693
 encoding utf-8
 Sheet 1 1
@@
 BS1
 $Comp
-L GND #PWR01
+L GND-RESCUE-adapter #PWR01
 U 1 1 5018FCBA
 P 12900 8450
 F 0 "#PWR01" H 12900 8450 30  0001 C CNN
 F 1 "GND" H 12900 8380 30  0001 C CNN
+F 2 "" H 12900 8450 60  0001 C CNN
+F 3 "" H 12900 8450 60  0001 C CNN
 	1    12900 8450
 	1    0    0    -1
@@
 	15150 3150 15600 3150
 $Comp
-L GND #PWR02
+L GND-RESCUE-adapter #PWR02
 U 1 1 5017B319
 P 12800 4300
 F 0 "#PWR02" H 12800 4300 30  0001 C CNN
 F 1 "GND" H 12800 4230 30  0001 C CNN
+F 2 "" H 12800 4300 60  0001 C CNN
+F 3 "" H 12800 4300 60  0001 C CNN
 	1    12800 4300
 	1    0    0    -1
@@
 F 1 "ATTINY84-P" H 14600 7000 60  0000 C CNN
 F 2 "DIP14" H 13350 7000 60  0001 C CNN
+F 3 "" H 14050 7750 60  0001 C CNN
 	1    14050 7750
 	1    0    0    -1
@@
 F 1 "ATMEGA16M1-M" H 14350 1550 50  0000 L BNN
 F 2 "QFN32" H 13300 1600 50  0001 C CNN
+F 3 "" H 14050 2950 60  0001 C CNN
 	1    14050 2950
 	1    0    0    -1
@@
 VCC
 $Comp
-L GND #PWR03
+L GND-RESCUE-adapter #PWR03
 U 1 1 5016C700
 P 10300 6150
 F 0 "#PWR03" H 10300 6150 30  0001 C CNN
 F 1 "GND" H 10300 6080 30  0001 C CNN
+F 2 "" H 10300 6150 60  0001 C CNN
+F 3 "" H 10300 6150 60  0001 C CNN
 	1    10300 6150
 	1    0    0    -1
 $EndComp
 $Comp
-L CPSMALL C4
+L CPsmall C4
 U 1 1 5016C6FF
 P 10300 5950
 F 0 "C4" H 10325 6000 30  0000 L CNN
 F 1 "10nF" H 10325 5875 30  0000 L CNN
+F 2 "" H 10300 5950 60  0001 C CNN
+F 3 "" H 10300 5950 60  0001 C CNN
 	1    10300 5950
 	1    0    0    -1
 $EndComp
 $Comp
-L CPSMALL C2
+L CPsmall C2
 U 1 1 5016C6B4
 P 6650 6400
 F 0 "C2" H 6675 6450 30  0000 L CNN
 F 1 "10nF" H 6675 6325 30  0000 L CNN
+F 2 "" H 6650 6400 60  0001 C CNN
+F 3 "" H 6650 6400 60  0001 C CNN
 	1    6650 6400
 	1    0    0    -1
 $EndComp
 $Comp
-L GND #PWR04
+L GND-RESCUE-adapter #PWR04
 U 1 1 5016C6B3
 P 6650 6600
 F 0 "#PWR04" H 6650 6600 30  0001 C CNN
 F 1 "GND" H 6650 6530 30  0001 C CNN
+F 2 "" H 6650 6600 60  0001 C CNN
+F 3 "" H 6650 6600 60  0001 C CNN
 	1    6650 6600
 	1    0    0    -1
@@
 VCC
 $Comp
-L CPSMALL C3
+L CPsmall C3
 U 1 1 5016C48B
 P 3300 3400
 F 0 "C3" H 3325 3450 30  0000 L CNN
 F 1 "10nF" H 3325 3325 30  0000 L CNN
+F 2 "" H 3300 3400 60  0001 C CNN
+F 3 "" H 3300 3400 60  0001 C CNN
 	1    3300 3400
 	1    0    0    -1
 $EndComp
 $Comp
-L GND #PWR05
+L GND-RESCUE-adapter #PWR05
 U 1 1 5016C48A
 P 3300 3600
 F 0 "#PWR05" H 3300 3600 30  0001 C CNN
 F 1 "GND" H 3300 3530 30  0001 C CNN
+F 2 "" H 3300 3600 60  0001 C CNN
+F 3 "" H 3300 3600 60  0001 C CNN
 	1    3300 3600
 	1    0    0    -1
@@
 VCC
 $Comp
-L GND #PWR06
+L GND-RESCUE-adapter #PWR06
 U 1 1 5016C3EB
 P 9950 3400
 F 0 "#PWR06" H 9950 3400 30  0001 C CNN
 F 1 "GND" H 9950 3330 30  0001 C CNN
+F 2 "" H 9950 3400 60  0001 C CNN
+F 3 "" H 9950 3400 60  0001 C CNN
 	1    9950 3400
 	1    0    0    -1
@@
 BS2
 $Comp
-L ATTINY15-P-GOOD IC7
+L ATTINY15-P-good IC7
 U 1 1 50169663
 P 7250 8600
@@
 F 1 "ATTINY15-P-GOOD" H 8550 7850 60  0000 C CNN
 F 2 "DIP8" H 7350 7850 60  0001 C CNN
+F 3 "" H 7250 8600 60  0001 C CNN
 	1    7250 8600
 	1    0    0    -1
@@
 VCC
 $Comp
-L GND #PWR07
+L GND-RESCUE-adapter #PWR07
 U 1 1 50168CAB
 P 3300 8850
 F 0 "#PWR07" H 3300 8850 30  0001 C CNN
 F 1 "GND" H 3300 8780 30  0001 C CNN
+F 2 "" H 3300 8850 60  0001 C CNN
+F 3 "" H 3300 8850 60  0001 C CNN
 	1    3300 8850
 	1    0    0    -1
 $EndComp
 $Comp
-L CPSMALL C5
+L CPsmall C5
 U 1 1 50168B28
 P 3300 8650
 F 0 "C5" H 3325 8700 30  0000 L CNN
 F 1 "10nF" H 3325 8575 30  0000 L CNN
+F 2 "" H 3300 8650 60  0001 C CNN
+F 3 "" H 3300 8650 60  0001 C CNN
 	1    3300 8650
 	1    0    0    -1
 $EndComp
 $Comp
-L CPSMALL C6
+L CPsmall C6
 U 1 1 50168AFA
 P 9950 3200
 F 0 "C6" H 9975 3250 30  0000 L CNN
 F 1 "10nF" H 9975 3125 30  0000 L CNN
+F 2 "" H 9950 3200 60  0001 C CNN
+F 3 "" H 9950 3200 60  0001 C CNN
 	1    9950 3200
 	1    0    0    -1
@@
 CLK
 $Comp
-L GND #PWR08
+L GND-RESCUE-adapter #PWR08
 U 1 1 50166675
 P 6800 1900
 F 0 "#PWR08" H 6800 1900 30  0001 C CNN
 F 1 "GND" H 6800 1830 30  0001 C CNN
+F 2 "" H 6800 1900 60  0001 C CNN
+F 3 "" H 6800 1900 60  0001 C CNN
 	1    6800 1900
 	1    0    0    -1
 $EndComp
 $Comp
-L GND #PWR09
+L GND-RESCUE-adapter #PWR09
 U 1 1 501664B7
 P 8000 7100
 F 0 "#PWR09" H 8000 7100 30  0001 C CNN
 F 1 "GND" H 8000 7030 30  0001 C CNN
+F 2 "" H 8000 7100 60  0001 C CNN
+F 3 "" H 8000 7100 60  0001 C CNN
 	1    8000 7100
 	1    0    0    -1
 $EndComp
 $Comp
-L GND #PWR010
+L GND-RESCUE-adapter #PWR010
 U 1 1 50166453
 P 7800 4100
 F 0 "#PWR010" H 7800 4100 30  0001 C CNN
 F 1 "GND" H 7800 4030 30  0001 C CNN
+F 2 "" H 7800 4100 60  0001 C CNN
+F 3 "" H 7800 4100 60  0001 C CNN
 	1    7800 4100
 	1    0    0    -1
 $EndComp
 $Comp
-L GND #PWR011
+L GND-RESCUE-adapter #PWR011
 U 1 1 5016640D
 P 10650 6800
 F 0 "#PWR011" H 10650 6800 30  0001 C CNN
 F 1 "GND" H 10650 6730 30  0001 C CNN
+F 2 "" H 10650 6800 60  0001 C CNN
+F 3 "" H 10650 6800 60  0001 C CNN
 	1    10650 6800
 	1    0    0    -1
 $EndComp
 $Comp
-L GND #PWR012
+L GND-RESCUE-adapter #PWR012
 U 1 1 501663FB
 P 12550 9300
 F 0 "#PWR012" H 12550 9300 30  0001 C CNN
 F 1 "GND" H 12550 9230 30  0001 C CNN
+F 2 "" H 12550 9300 60  0001 C CNN
+F 3 "" H 12550 9300 60  0001 C CNN
 	1    12550 9300
 	1    0    0    -1
 $EndComp
 $Comp
-L GND #PWR013
+L GND-RESCUE-adapter #PWR013
 U 1 1 501663EF
 P 9150 9300
 F 0 "#PWR013" H 9150 9300 30  0001 C CNN
 F 1 "GND" H 9150 9230 30  0001 C CNN
+F 2 "" H 9150 9300 60  0001 C CNN
+F 3 "" H 9150 9300 60  0001 C CNN
 	1    9150 9300
 	1    0    0    -1
 $EndComp
 $Comp
-L GND #PWR014
+L GND-RESCUE-adapter #PWR014
 U 1 1 501663DB
 P 4500 10550
 F 0 "#PWR014" H 4500 10550 30  0001 C CNN
 F 1 "GND" H 4500 10480 30  0001 C CNN
+F 2 "" H 4500 10550 60  0001 C CNN
+F 3 "" H 4500 10550 60  0001 C CNN
 	1    4500 10550
 	1    0    0    -1
 $EndComp
 $Comp
-L GND #PWR015
+L GND-RESCUE-adapter #PWR015
 U 1 1 501663BC
 P 4300 5150
 F 0 "#PWR015" H 4300 5150 30  0001 C CNN
 F 1 "GND" H 4300 5080 30  0001 C CNN
+F 2 "" H 4300 5150 60  0001 C CNN
+F 3 "" H 4300 5150 60  0001 C CNN
 	1    4300 5150
 	1    0    0    -1
 $EndComp
 $Comp
-L GND #PWR016
+L GND-RESCUE-adapter #PWR016
 U 1 1 501663AC
 P 900 5350
 F 0 "#PWR016" H 900 5350 30  0001 C CNN
 F 1 "GND" H 900 5280 30  0001 C CNN
+F 2 "" H 900 5350 60  0001 C CNN
+F 3 "" H 900 5350 60  0001 C CNN
 	1    900  5350
 	1    0    0    -1
@@
 F 0 "P1" H 2250 6300 60  0000 C CNN
 F 1 "CONN_10X2" V 2250 5650 50  0000 C CNN
+F 2 "" H 2250 5750 60  0001 C CNN
+F 3 "" H 2250 5750 60  0001 C CNN
 	1    2250 5750
 	1    0    0    -1
 $EndComp
 $Comp
-L ATTINY26-P IC4
+L ATTINY26-P-RESCUE-adapter IC4
 U 1 1 50165155
 P 11550 5900
@@
 F 1 "ATTINY26-P" H 11850 4950 60  0000 C CNN
 F 2 "DIP20" H 11100 4950 60  0001 C CNN
+F 3 "" H 11550 5900 60  0001 C CNN
 	1    11550 5900
 	1    0    0    -1
 $EndComp
 $Comp
-L ATTINY11-P IC8
+L ATTINY11-P-RESCUE-adapter IC8
 U 1 1 50164FFE
 P 10650 8600
@@
 F 1 "ATTINY11-P" H 11950 7850 60  0000 C CNN
 F 2 "DIP8" H 10750 7850 60  0001 C CNN
+F 3 "" H 10650 8600 60  0001 C CNN
 	1    10650 8600
 	1    0    0    -1
 $EndComp
 $Comp
-L ATTINY2313-P IC2
+L ATTINY2313-P-RESCUE-adapter IC2
 U 1 1 50164F39
 P 8000 6000
@@
 F 1 "ATTINY2313-P" H 8600 5150 60  0000 C CNN
 F 2 "DIP20" H 7200 5150 60  0001 C CNN
+F 3 "" H 8000 6000 60  0001 C CNN
 	1    8000 6000
 	1    0    0    -1
@@
 F 1 "ATMEGA8-P" H 8150 1100 50  0000 L BNN
 F 2 "DIL28" H 7200 1150 50  0001 C CNN
+F 3 "" H 7800 2500 60  0001 C CNN
 	1    7800 2500
 	1    0    0    -1
 $EndComp
 $Comp
-L AT90S8515-P IC5
+L AT90S8515-P-RESCUE-adapter IC5
 U 1 1 50164BA2
 P 4500 8450
@@
 F 1 "AT90S8515-P" H 4750 6550 50  0000 L BNN
 F 2 "DIL40" H 3800 6600 50  0001 C CNN
+F 3 "" H 4500 8450 60  0001 C CNN
 	1    4500 8450
 	1    0    0    -1
@@
 F 1 "ATMEGA16-P" H 4650 1150 50  0000 L BNN
 F 2 "DIL40" H 3650 1200 50  0001 C CNN
+F 3 "" H 4350 3050 60  0001 C CNN
 	1    4350 3050
 	1    0    0    -1
