File: circuit/fuser-32/hvpp.sch (KiCad schematic (older format))
At the start: 66 parts, among them CON1 AVR-ISP-10, IC1 ATMEGA32-P, J1 USB, P1 CONN_10X2, Q1 BC337, Q2 BC847, Q3 BC857, Q4 BC847, Q5 BC857, X1 16MHz

Commit message: fuser-32 programmer PCB: open with kicad 4.x and saving
Parts:
- C1, C2: symbol C -> C-RESCUE-hvpp
- C3, C6: symbol CSMALL -> Csmall
- C4, C5: symbol CPSMALL -> CPsmall
- D3: symbol LED -> LED-RESCUE-hvpp
- R1, R10, R11, R12, R13, R14, R15, R16, R17, R18, R19, R2, R20, R21, R22, R24, R25, R26, R27, R28, R29, R3, R30, R31, R32, R33, R34, R35, R36, R37, R38, R39, R4, R5, R6, R7, R8, R9: symbol R -> R-RESCUE-hvpp
Changed lines of the file:
@@
 EESchema Schematic File Version 2
+LIBS:hvpp-rescue
 LIBS:power
 LIBS:device
@@
 LIBS:memory
 LIBS:xilinx
-LIBS:special
 LIBS:microcontrollers
 LIBS:dsp
@@
 LIBS:dual-led
 LIBS:hvpp-cache
-EELAYER 27 0
+EELAYER 25 0
 EELAYER END
 $Descr A4 11693 8268
@@
 	10750 3000 11150 3000
 $Comp
-L R R32
+L R-RESCUE-hvpp R32
 U 1 1 5072CEC6
 P 10500 2300
@@
 $EndComp
 $Comp
-L R R34
+L R-RESCUE-hvpp R34
 U 1 1 5072CEC5
 P 10500 2500
@@
 $EndComp
 $Comp
-L R R33
+L R-RESCUE-hvpp R33
 U 1 1 5072CEC4
 P 10500 2400
@@
 $EndComp
 $Comp
-L R R36
+L R-RESCUE-hvpp R36
 U 1 1 5072CEC3
 P 10500 2700
@@
 $EndComp
 $Comp
-L R R37
+L R-RESCUE-hvpp R37
 U 1 1 5072CEC2
 P 10500 2800
@@
 $EndComp
 $Comp
-L R R35
+L R-RESCUE-hvpp R35
 U 1 1 5072CEC1
 P 10500 2600
@@
 $EndComp
 $Comp
-L R R38
+L R-RESCUE-hvpp R38
 U 1 1 5072CEC0
 P 10500 2900
@@
 $EndComp
 $Comp
-L R R39
+L R-RESCUE-hvpp R39
 U 1 1 5072CEBE
 P 10500 3000
@@
 	7700 2900 8100 2900
 $Comp
-L R R30
+L R-RESCUE-hvpp R30
 U 1 1 5072CE8D
 P 8350 2900
@@
 $EndComp
 $Comp
-L R R31
+L R-RESCUE-hvpp R31
 U 1 1 5072CE8C
 P 8350 3000
@@
 	7700 2800 8100 2800
 $Comp
-L R R29
+L R-RESCUE-hvpp R29
 U 1 1 5072CE8B
 P 8350 2800
@@
 $EndComp
 $Comp
-L R R26
+L R-RESCUE-hvpp R26
 U 1 1 5072CE84
 P 8350 2500
@@
 	7700 2700 8100 2700
 $Comp
-L R R28
+L R-RESCUE-hvpp R28
 U 1 1 5072CE83
 P 8350 2700
@@
 $EndComp
 $Comp
-L R R27
+L R-RESCUE-hvpp R27
 U 1 1 5072CE82
 P 8350 2600
@@
 	7700 2300 8100 2300
 $Comp
-L R R24
+L R-RESCUE-hvpp R24
 U 1 1 5072CE75
 P 8350 2300
@@
 $EndComp
 $Comp
-L R R25
+L R-RESCUE-hvpp R25
 U 1 1 5072CE6D
 P 8350 2400
@@
 	5150 5850 5400 5850
 $Comp
-L R R21
+L R-RESCUE-hvpp R21
 U 1 1 5072CDDD
 P 4900 5850
@@
 $EndComp
 $Comp
-L R R22
+L R-RESCUE-hvpp R22
 U 1 1 5072CDC2
 P 4900 6050
@@
 $EndComp
 $Comp
-L R R20
+L R-RESCUE-hvpp R20
 U 1 1 5072CDB6
 P 4900 5650
@@
 MOSI_A
 $Comp
-L CSMALL C6
+L Csmall C6
 U 1 1 50326F5F
 P 6000 2750
@@
 nVCC
 $Comp
-L R R19
+L R-RESCUE-hvpp R19
 U 1 1 502BA262
 P 8550 6100
@@
 RDY
 $Comp
-L CSMALL C3
+L Csmall C3
 U 1 1 50200892
 P 6050 7350
@@
 $EndComp
 $Comp
-L GND #PWR03
+L GND-RESCUE-hvpp #PWR03
 U 1 1 5020085E
 P 6050 7500
@@
 $EndComp
 $Comp
-L GND #PWR04
+L GND-RESCUE-hvpp #PWR04
 U 1 1 50141AEF
 P 700 7050
@@
 LEDG
 $Comp
-L GND #PWR05
+L GND-RESCUE-hvpp #PWR05
 U 1 1 5013D2F2
 P 6550 3450
@@
 TXD_A
 $Comp
-L GND #PWR06
+L GND-RESCUE-hvpp #PWR06
 U 1 1 50108CCA
 P 5650 3250
@@
 $EndComp
 $Comp
-L R R18
+L R-RESCUE-hvpp R18
 U 1 1 50108C9E
 P 5650 2000
@@
 SCK_A
 $Comp
-L R R17
+L R-RESCUE-hvpp R17
 U 1 1 50108C41
 P 4900 5950
@@
 $EndComp
 $Comp
-L R R16
+L R-RESCUE-hvpp R16
 U 1 1 50091466
 P 6450 2200
@@
 VCC
 $Comp
-L GND #PWR07
+L GND-RESCUE-hvpp #PWR07
 U 1 1 5006947D
 P 7450 2150
@@
 RST
 $Comp
-L GND #PWR08
+L GND-RESCUE-hvpp #PWR08
 U 1 1 50068018
 P 3600 7500
@@
 $EndComp
 $Comp
-L R R12
+L R-RESCUE-hvpp R12
 U 1 1 50068006
 P 3600 6050
@@
 $EndComp
 $Comp
-L R R14
+L R-RESCUE-hvpp R14
 U 1 1 50067B6D
 P 8550 5800
@@
 $EndComp
 $Comp
-L R R15
+L R-RESCUE-hvpp R15
 U 1 1 50067B6B
 P 10100 4900
@@
 CLK
 $Comp
-L R R13
+L R-RESCUE-hvpp R13
 U 1 1 500593DA
 P 4900 5750
@@
 $EndComp
 $Comp
-L GND #PWR09
+L GND-RESCUE-hvpp #PWR09
 U 1 1 50059324
 P 6150 5800
@@
 RXD
 $Comp
-L R R11
+L R-RESCUE-hvpp R11
 U 1 1 500591F1
 P 6400 6050
@@
 $EndComp
 $Comp
-L R R10
+L R-RESCUE-hvpp R10
 U 1 1 500591D2
 P 6400 5950
@@
 $EndComp
 $Comp
-L R R9
+L R-RESCUE-hvpp R9
 U 1 1 500590F9
 P 3600 5450
@@
 $EndComp
 $Comp
-L R R8
+L R-RESCUE-hvpp R8
 U 1 1 500580E3
 P 9500 4800
@@
 $EndComp
 $Comp
-L R R3
+L R-RESCUE-hvpp R3
 U 1 1 500580CA
 P 9500 4650
@@
 $EndComp
 $Comp
-L CPSMALL C4
+L CPsmall C4
 U 1 1 4FBD6717
 P 8550 4800
@@
 $EndComp
 $Comp
-L R R5
+L R-RESCUE-hvpp R5
 U 1 1 4FBD637C
 P 1950 6350
@@
 $EndComp
 $Comp
-L GND #PWR013
+L GND-RESCUE-hvpp #PWR013
 U 1 1 4FBD635C
 P 2100 7400
@@
 $EndComp
 $Comp
-L GND #PWR014
+L GND-RESCUE-hvpp #PWR014
 U 1 1 4FBD6359
 P 1950 7400
@@
 $EndComp
 $Comp
-L R R7
+L R-RESCUE-hvpp R7
 U 1 1 4FBD631D
 P 2450 6700
@@
 $EndComp
 $Comp
-L R R6
+L R-RESCUE-hvpp R6
 U 1 1 4FBD630F
 P 2450 6850
@@
 $EndComp
 $Comp
-L GND #PWR015
+L GND-RESCUE-hvpp #PWR015
 U 1 1 4FBD62F1
 P 1650 7050
@@
 LEDRED
 $Comp
-L R R2
+L R-RESCUE-hvpp R2
 U 1 1 4FBD61F9
 P 6650 2200
@@
 $EndComp
 $Comp
-L CPSMALL C5
+L CPsmall C5
 U 1 1 4FBD615C
 P 6550 7350
@@
 $EndComp
 $Comp
-L GND #PWR017
+L GND-RESCUE-hvpp #PWR017
 U 1 1 4FBD6145
 P 6550 7500
@@
 RESET
 $Comp
-L GND #PWR019
+L GND-RESCUE-hvpp #PWR019
 U 1 1 4FBD5E96
 P 650 1800
@@
 $EndComp
 $Comp
-L C C1
+L C-RESCUE-hvpp C1
 U 1 1 4FBD5E87
 P 1000 1350
@@
 $EndComp
 $Comp
-L C C2
+L C-RESCUE-hvpp C2
 U 1 1 4FBD5E82
 P 1000 2050
@@
 $EndComp
 $Comp
-L LED D3
+L LED-RESCUE-hvpp D3
 U 1 1 4FBD5D47
 P 8350 4600
@@
 RSTH
 $Comp
-L R R4
+L R-RESCUE-hvpp R4
 U 1 1 4FAFC417
 P 8550 5650
@@
 $EndComp
 $Comp
-L GND #PWR021
+L GND-RESCUE-hvpp #PWR021
 U 1 1 4FAF901B
 P 2450 4800
@@
 PWM
 $Comp
-L GND #PWR025
+L GND-RESCUE-hvpp #PWR025
 U 1 1 4FAF8F74
 P 7950 5450
@@
 $EndComp
 $Comp
-L GND #PWR026
+L GND-RESCUE-hvpp #PWR026
 U 1 1 4FAF8F6D
 P 2350 4800
@@
 $EndComp
 $Comp
-L R R1
+L R-RESCUE-hvpp R1
 U 1 1 4FAF8E67
 P 7000 4800
